File: kicad/FreqCounter32v203.kicad_pcb (KiCad board)
At the start: 2 copper layers, 30 x 40 mm, 34 parts, among them J1 max4466_Mic_Module, J2 WCH-LINKE, J3 Conn_01x07_Socket, SW1 OK, SW2 ↓, SW3 ↑, SW7 SWITCH_INV, U1 SEEED_GROVE, U3 CH32V003F4P6, U4 XC6206PxxxMR, U5 USB-C_16PIN, Y1 24M

Commit message: in progress
Parts:
- removed STAND: MountingHole_3mm, MountingHole:MountingHole_3mm
- added C10: 0.1, Capacitor_SMD:C_0402_1005Metric, F.Cu at (96.2, 44.2)
- added C11: 10u, Capacitor_SMD:C_0402_1005Metric, F.Cu at (96.2, 46.2)
- added C12: 0.1u, Capacitor_SMD:C_0402_1005Metric, F.Cu at (96.2, 48.1)
- added C14: 10u, Capacitor_THT:CP_Radial_D5.0mm_P2.50mm, F.Cu at (87.3, 53.0)
- added C15: 0.1, Capacitor_SMD:C_0402_1005Metric, F.Cu at (96.2, 50.1)
- added C7: 20p, Capacitor_SMD:C_0603_1608Metric, F.Cu at (75.0, 73.7)
- added C8: 20p, Capacitor_SMD:C_0603_1608Metric, F.Cu at (75.0, 76.2)
- added C9: 10u, Capacitor_THT:CP_Radial_D5.0mm_P2.50mm, F.Cu at (87.3, 46.5)
- added FB1: FerriteBead_Small, Capacitor_SMD:C_0402_1005Metric, F.Cu at (96.2, 52.1)
- added FB2: FerriteBead_Small, Capacitor_SMD:C_0402_1005Metric, F.Cu at (99.0, 44.2)
- added FB3: FerriteBead_Small, Capacitor_SMD:C_0402_1005Metric_Pad0.74x0.62mm_HandSolder, F.Cu at (98.5, 33.9)
- added FB4: FerriteBead_Small, Capacitor_SMD:C_0402_1005Metric, F.Cu at (99.0, 46.2)
- added J4: AKBONE2024_SOCKET, Connector_PinSocket_2.54mm:PinSocket_1x13_P2.54mm_Vertical, F.Cu at (127.6, 31.7)
- added MK1: mic, Capacitor_THT:CP_Radial_Tantal_D6.0mm_P2.50mm, F.Cu at (130.1, 75.2)
- added MK2: mic, Capacitor_THT:CP_Radial_Tantal_D6.0mm_P2.50mm, F.Cu at (157.6, 75.2)
- added Q1: NMOS LX2302S, Package_TO_SOT_SMD:SOT-23, F.Cu at (81.1, 75.6)
- added Q2: PMOS_GSD_RC2101, Package_TO_SOT_SMD:SOT-323_SC-70, F.Cu at (99.1, 31.1)
- added R10: 5.1k, Resistor_SMD:R_0402_1005Metric, F.Cu at (89.6, 32.3)
- added R11: 5.1k, Resistor_SMD:R_0402_1005Metric, F.Cu at (89.6, 34.3)
- added R12: 1.5k, Resistor_SMD:R_0402_1005Metric, F.Cu at (89.6, 36.2)
- added R13: 47, Resistor_SMD:R_0402_1005Metric, F.Cu at (89.6, 38.2)
- added R14: 47, Resistor_SMD:R_0402_1005Metric, F.Cu at (89.6, 40.2)
- added R15: 1k, Resistor_SMD:R_0402_1005Metric, F.Cu at (89.6, 42.2)
- added R16: 10k, Resistor_SMD:R_0402_1005Metric, F.Cu at (92.5, 30.3)
- added R17: 10k, Resistor_SMD:R_0402_1005Metric, F.Cu at (92.5, 32.3)
- added R18: 59k, Resistor_SMD:R_0402_1005Metric, F.Cu at (92.5, 34.3)
- added R19: 1k, Resistor_SMD:R_0402_1005Metric, F.Cu at (92.5, 36.2)
- added R20: 1k, Resistor_SMD:R_0402_1005Metric, F.Cu at (92.5, 38.2)
- added R21: 1k, Resistor_SMD:R_0402_1005Metric, F.Cu at (92.5, 40.2)
- added R22: 59k, Resistor_SMD:R_0402_1005Metric, F.Cu at (92.5, 42.2)
- added R23: 3.3k, Resistor_SMD:R_0402_1005Metric, F.Cu at (95.4, 30.3)
- added R24: 12k, Resistor_SMD:R_0402_1005Metric, F.Cu at (95.4, 32.3)
- added R25: 4.7k, Resistor_SMD:R_0402_1005Metric, F.Cu at (95.4, 34.3)
- added REF**: MountingHole_2.2mm_M2, MountingHole:MountingHole_2.2mm_M2, F.Cu at (131.1, 66.2)
- added REF**: MountingHole_2.2mm_M2, MountingHole:MountingHole_2.2mm_M2, F.Cu at (155.1, 66.2)
- added RV1: 200k, Potentiometer_THT:Potentiometer_ACP_CA9-H2,5_Horizontal, F.Cu at (140.1, 72.2)
- added RV2: 200k, Potentiometer_THT:Potentiometer_ACP_CA9-H2,5_Horizontal, F.Cu at (150.6, 72.2)
- added U2: OLED_0.96in_SPI, library:OLED_0.96in_SPI, F.Cu at (41.4, 48.7)
- added U6: CH32C203C8T6, Package_DFN_QFN:Infineon_MLPQ-48-1EP_7x7mm_P0.5mm_EP5.15x5.15mm, F.Cu at (144.6, 47.9)
- added U7: LMV358, Package_SO:SSOP-8_2.95x2.8mm_P0.65mm, F.Cu at (142.9, 66.3)
- added Y2: 32.768k, Crystal:Crystal_DS15_D1.5mm_L5.0mm_Vertical, F.Cu at (137.4, 45.7)
- C1, C2, C4, C5, C6: footprint Capacitor_SMD:C_0603_1608Metric -> Capacitor_SMD:C_0402_1005Metric
- J1: value max4466_Mic_Module -> BOOT; footprint Connector_PinHeader_2.54mm:PinHeader_1x03_P2.54mm_Vertical -> Connector_PinSocket_2.54mm:PinSocket_2x03_P2.54mm_Vertical
- J2: value WCH-LINKE -> WCH_LINK; footprint Connector_PinHeader_2.54mm:PinHeader_1x06_P2.54mm_Vertical -> Capacitor_SMD:C_0402_1005Metric; moved to F.Cu
- R1, R2, R3, R4, R5, R6, R7, R8, R9: footprint Resistor_SMD:R_0603_1608Metric -> Resistor_SMD:R_0402_1005Metric
- SW1, SW2, SW3: footprint Button_Switch_SMD:SW_Push_1P1T_NO_6x6mm_H9.5mm -> Button_Switch_THT:SW_SPST_Omron_B3F-315x_Angled
- U3: value CH32V003F4P6 -> USB-C_16PIN; footprint Package_SO:TSSOP-20_4.4x6.5mm_P0.65mm -> library:USB_Type_C_16Pin_Female
- Y1: value 24M -> 32M; footprint Crystal:Crystal_SMD_HC49-SD -> Crystal:Crystal_DS15_D1.5mm_L5.0mm_Vertical; moved to F.Cu
- moved R1 69.7 mm to (86.7, 30.3)
- moved C3 65.1 mm to (75.0, 71.2)
- moved R5 62.3 mm to (86.7, 36.2), turned to 0 degrees
- moved C6 58.9 mm to (93.3, 52.1)
- moved C5 57.9 mm to (93.3, 50.1)
- moved C4 56.6 mm to (93.3, 48.1)
- moved R6 55.5 mm to (86.7, 38.2), turned to 0 degrees
- moved R3 55.4 mm to (86.7, 34.3)
- moved R2 55.2 mm to (86.7, 32.3)
- moved R9 51.1 mm to (89.6, 30.3), turned to 0 degrees
- moved R7 50.9 mm to (86.7, 40.2), turned to 0 degrees
- moved R8 50.2 mm to (86.7, 42.2), turned to 0 degrees
- moved C1 46.0 mm to (93.3, 44.2), turned to 0 degrees
- moved C2 43.5 mm to (93.3, 46.2)
- moved J2 32.2 mm to (99.0, 48.1), turned to 0 degrees
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Connections:
- BT1 pad 1: Net-(BT1-Pad1) -> BATT
- BT1 pad 2: GND -> AGND
- C1 pad 1: +3V3 -> VCC
- C2 pad 2: Net-(U3-PA1/OSCI/A1/T1CH2/OPN0) -> Net-(U6-OSC_IN/PD0)
- C3 pad 2: Net-(U3-PA2/OSCO/A0/T1CH2N/OPP0/AETR2_) -> Net-(U6-OSC_OUT/PD1)
- C4 pad 1: +3V3 -> AVCC
- C4 pad 2: GND -> AGND
- C6 pad 2: +3V3 -> Net-(Q1-D)
- J1 pad 1: Net-(J1-Pin_1) -> VCC
- J1 pad 2: GND -> BOOT0
- J1 pad 3: +3V3 -> GND
- J2 pad 1: +3V3 -> VCC
- J3 pad 2: +3V3 -> VCC
- J3 pad 3: Net-(J3-Pin_3) -> SCK
- J3 pad 4: Net-(J3-Pin_4) -> MOSI
- J3 pad 5: Net-(J3-Pin_5) -> OLED_RESET
- J3 pad 6: Net-(J3-Pin_6) -> DC
- J3 pad 7: Net-(J3-Pin_7) -> CS
- JP1 pad 1: Net-(JP1-A) -> SPEAKER
- R1 pad 1: Net-(J2-Pin_5) -> LED
- R2 pad 1: +3V3 -> VCC
- R4 pad 1: Net-(JP1-A) -> SPEAKER
- R7 pad 1: +3V3 -> Net-(U5-DN1)
- R7 pad 2: Net-(U5-DN1) -> VCC
- R8 pad 2: Net-(U3-PA1/OSCI/A1/T1CH2/OPN0) -> USB1_DP
- R9 pad 2: Net-(U3-PA2/OSCO/A0/T1CH2N/OPP0/AETR2_) -> USB1_DN
- SW7 pad 1: Net-(BT1-Pad1) -> Net-(Q2-S)
- SW7 pad 2: +3V3 -> AVCC
- U1 pad 3: +3V3 -> VCC
- U4 pad 2: +3V3 -> Net-(Q1-D)
- U5 pad A4: +5V -> Net-(FB4-Pad1)
- U5 pad B9: +5V -> Net-(FB4-Pad1)
- Y1 pad 1: Net-(U3-PA2/OSCO/A0/T1CH2N/OPP0/AETR2_) -> Net-(U6-OSC_OUT/PD1)
- Y1 pad 2: Net-(U3-PA1/OSCI/A1/T1CH2/OPN0) -> Net-(U6-OSC_IN/PD0)
Routing:
- net GND: track 162.5 -> 0.00 mm, vias 9 -> 0
- net Net-(BT1-Pad1): track 89.5 -> 0.00 mm
- net +3V3: track 88.3 -> 0.00 mm
- net Net-(R2-Pad2): track 51.0 -> 0.00 mm, vias 2 -> 0
- net SW3: track 40.9 -> 0.00 mm, vias 4 -> 0
- net Net-(J2-Pin_5): track 39.5 -> 0.00 mm, vias 3 -> 0
- net SW1: track 31.3 -> 0.00 mm, vias 2 -> 0
- net Net-(U5-DP1): track 26.8 -> 0.00 mm, vias 2 -> 0
- net SW2: track 24.3 -> 0.00 mm
- net +5V: track 23.9 -> 0.00 mm
- net Net-(J2-Pin_2): track 23.5 -> 0.00 mm, vias 1 -> 0
- net Net-(J2-Pin_6): track 21.7 -> 0.00 mm, vias 2 -> 0
- net Net-(U5-DN1): track 21.5 -> 0.00 mm, vias 2 -> 0
- net Net-(J3-Pin_3): track 18.5 -> 0.00 mm, vias 1 -> 0
- net Net-(J2-Pin_4): track 17.0 -> 0.00 mm, vias 2 -> 0
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Other:
- board size 30 x 40 mm -> 35 x 40 mm
