File: kicad/FreqCounter32v203.kicad_sch (KiCad schematic)
At the start: 32 parts, among them J1 max4466_Mic_Module, J2 WCH-LINKE, J3 Conn_01x07_Socket, SW1 OK, SW2 ↓, SW3 ↑, SW7 SWITCH_INV, U1 SEEED_GROVE, U2 OLED_0.96in_SPI, U3 CH32V003F4P6, U4 XC6206PxxxMR, U5 USB-C_16PIN, Y1 24M

Commit message: in progress
Parts:
- removed J1: max4466_Mic_Module, Connector_PinHeader_2.54mm:PinHeader_1x03_P2.54mm_Vertical, symbol Connector:Conn_01x03_Socket
- removed J2: WCH-LINKE, Connector_PinHeader_2.54mm:PinHeader_1x06_P2.54mm_Vertical, symbol Connector:Conn_01x06_Pin
- removed U3: CH32V003F4P6, Package_SO:TSSOP-20_4.4x6.5mm_P0.65mm, symbol nanbuwks:CH32V003F4P6
- added C10, C15: 0.1, Capacitor_SMD:C_0402_1005Metric, symbol Device:C
- added C11: 10u, Capacitor_SMD:C_0402_1005Metric, symbol FreqCounter3203-rescue:C
- added C12: 0.1u, Capacitor_SMD:C_0402_1005Metric, symbol FreqCounter3203-rescue:C
- added C14, C9: 10u, Capacitor_THT:CP_Radial_D5.0mm_P2.50mm, symbol Device:C_Polarized
- added C7, C8: 20p, Capacitor_SMD:C_0603_1608Metric, symbol Device:C
- added FB1, FB2, FB4: FerriteBead_Small, Capacitor_SMD:C_0402_1005Metric, symbol Device:FerriteBead_Small
- added FB3: FerriteBead_Small, Capacitor_SMD:C_0402_1005Metric_Pad0.74x0.62mm_HandSolder, symbol Device:FerriteBead_Small
- added J1: BOOT, Connector_PinSocket_2.54mm:PinSocket_2x03_P2.54mm_Vertical, symbol Connector_Generic:Conn_02x03_Counter_Clockwise
- added J2: WCH_LINK, Capacitor_SMD:C_0402_1005Metric, symbol Connector:Conn_01x08_Pin
- added J4: AKBONE2024_SOCKET, Connector_PinSocket_2.54mm:PinSocket_1x13_P2.54mm_Vertical, symbol Connector:Conn_01x13_Socket
- added MK1, MK2: mic, Capacitor_THT:CP_Radial_Tantal_D6.0mm_P2.50mm, symbol Device:Microphone_Condenser
- added Q1: NMOS LX2302S, Package_TO_SOT_SMD:SOT-23, symbol Simulation_SPICE:NMOS
- added Q2: PMOS_GSD_RC2101, Package_TO_SOT_SMD:SOT-323_SC-70, symbol Device:Q_PMOS_GSD
- added R10, R11: 5.1k, Resistor_SMD:R_0402_1005Metric, symbol FreqCounter3203-rescue:R
- added R12: 1.5k, Resistor_SMD:R_0402_1005Metric, symbol FreqCounter3203-rescue:R
- added R13, R14: 47, Resistor_SMD:R_0402_1005Metric, symbol FreqCounter3203-rescue:R
- added R15, R19, R20, R21: 1k, Resistor_SMD:R_0402_1005Metric, symbol Device:R
- added R16, R17: 10k, Resistor_SMD:R_0402_1005Metric, symbol Device:R
- added R18, R22: 59k, Resistor_SMD:R_0402_1005Metric, symbol Device:R
- added R23: 3.3k, Resistor_SMD:R_0402_1005Metric, symbol Device:R
- added R24: 12k, Resistor_SMD:R_0402_1005Metric, symbol Device:R
- added R25: 4.7k, Resistor_SMD:R_0402_1005Metric, symbol Device:R
- added RV1, RV2: 200k, Potentiometer_THT:Potentiometer_ACP_CA9-H2,5_Horizontal, symbol Device:R_Potentiometer
- added U3: USB-C_16PIN, library:USB_Type_C_16Pin_Female, symbol nanbuwks:USB-C_16PIN
- added U6: CH32C203C8T6, Package_DFN_QFN:Infineon_MLPQ-48-1EP_7x7mm_P0.5mm_EP5.15x5.15mm, symbol nanbuwks:CH32V203CxU6
- added U7: LMV358, Package_SO:SSOP-8_2.95x2.8mm_P0.65mm, symbol Amplifier_Operational:LMV358
- added Y2: 32.768k, Crystal:Crystal_DS15_D1.5mm_L5.0mm_Vertical, symbol Device:Crystal
- C1, C2, C4, C5, C6: footprint Capacitor_SMD:C_0603_1608Metric -> Capacitor_SMD:C_0402_1005Metric
- R1, R2, R3, R4, R5, R6, R7, R8, R9: footprint Resistor_SMD:R_0603_1608Metric -> Resistor_SMD:R_0402_1005Metric
- SW1, SW2, SW3: footprint Button_Switch_SMD:SW_Push_1P1T_NO_6x6mm_H9.5mm -> Button_Switch_THT:SW_SPST_Omron_B3F-315x_Angled
- Y1: value 24M -> 32M; footprint Crystal:Crystal_SMD_HC49-SD -> Crystal:Crystal_DS15_D1.5mm_L5.0mm_Vertical
Connections:
- net +3V3: now also R7.2, FB1.1, J1.1 (Pin_1), J1.6 (Pin_6), J2.1 (Pin_1), J4.1 (Pin_1), R12.2, U6.24 (VDD_VIO_1), U6.36 (VDD_2), U6.48 (VDD_VIO_3); no longer C4.1, C6.2, R7.1, SW7.2, U4.2 (VO)
- net +5V: now also FB3.2, FB4.2, U3.A9 (VBUS), U3.B4 (VBUS); no longer U5.A4 (VBUS), U5.B9 (VBUS)
- net GND: now also C7.1, C8.1, FB2.1, J1.3 (Pin_3), J1.4 (Pin_4), J2.4 (Pin_4), J2.6 (Pin_6), J4.2 (Pin_2), R10.2, R11.2, U3.A1 (GND), U3.A12 (GND), U3.B1 (GND), U3.B12 (GND), U6.0 (VSS), U6.23 (VSS_1), U6.35 (VSS_2), U6.47 (VSS_3); no longer BT1.2, C4.2
- net SW1: now also U6.18 (PB0/ADC8)
- net SW2: now also U6.19 (PB1/ADC9)
- net SW3: now also U6.39 (PB3)
- net at SW7.1: now also Q2.2 (S); no longer BT1.1
- net LED: now reaches R1.1
- net LED: now also U6.40 (PB4)
- net SCK: now reaches J3.3 (Pin_3), U2.3 (D0)
- net SCK: now also U6.15 (PA5/ADC5)
- net MOSI: now reaches J3.4 (Pin_4), U2.4 (D1)
- net MOSI: now also U6.17 (PA7/ADC7)
- net OLED_RESET: now reaches J3.5 (Pin_5), U2.5 (RST)
- net OLED_RESET: now also U6.29 (PA8)
- net DC: now reaches J3.6 (Pin_6), U2.6 (DC)
- net DC: now also U6.14 (PA4/ADC4)
- net CS: now reaches J3.7 (Pin_7), U2.7 (CS)
- net CS: now also U6.13 (PA3/ADC3)
- net at R9.1, U5.A7 (DN1), U5.B7 (DN2): now also R7.1; no longer R7.2
- net at C3.2, Y1.1: now also U6.6 (OSC_OUT/PD1); no longer R9.2
- net at C2.2, Y1.2: now also U6.5 (OSC_IN/PD0); no longer R8.2
- net SPEAKER: now reaches JP1.1 (A), R4.1
- net SPEAKER: now also U6.38 (PA15)
- net at U1.2 (White/Dn1/An1/TX/SDA): now also U6.46 (PB9)
- net at U1.1 (Yellow/Dn/An/RX/SCL): now also U6.45 (PB8)
- new net: J2.2 (Pin_2), U6.34 (PA13/SWDIO)
- new net: J2.3 (Pin_3), U6.37 (PA14/SWCLK)
- new net: J2.7 (Pin_7), U6.30 (PA9)
- new net: J2.8 (Pin_8), U6.31 (PA10)
- new net: R12.1, R13.1, U3.A7 (DN1), U3.B7 (DN2)
- new net: C7.2, U6.3 (PC14/OSC32IN), Y2.2
- new net: C8.2, U6.4 (PC15/OSC32OUT), Y2.1
- new net: C14.2, C15.1
- new net: FB4.1, U5.A4 (VBUS), U5.B9 (VBUS)
- new net: C14.1, MK2.2 (+), R19.2
- new net: C11.1, R23.1, R24.2, R25.1
- new net: R14.1, U3.A6 (DP1), U3.B6 (DP2)
- new net: FB3.1, U3.A4 (VBUS), U3.B9 (VBUS)
- new net: Q1.2 (G), R23.2
- new net: C6.2, FB1.2, Q1.1 (D), R25.2, U4.2 (VO)
- new net: R18.1, R21.2, U7.2 (-)
- new net: R18.2, RV1.1
- new net: R22.2, RV2.1
- new net: R11.1, U3.B5 (CC2)
- new net: C9.1, MK1.2 (+), R15.2
- new net: C10.1, C9.2
- new net: R20.2, R22.1, U7.6 (-)
- new net: R10.1, U3.A5 (CC1)
- new net ACENTER: J4.11 (Pin_11), R16.2, R17.1, R20.1, R21.1, U6.12 (PA2/ADC2)
- new net AGND: BT1.2, C11.2, C12.2, C4.2, FB2.2, J4.13 (Pin_13), MK1.1 (-), MK2.1 (-), Q2.1 (G), R17.2, R24.1, U6.8 (VSSA), U7.4 (V-)
- new net AVCC: C12.1, C4.1, Q1.3 (S), R15.1, R16.1, R19.1, SW7.2, U6.9 (VDDA), U7.8 (V+)
- new net BATT: BT1.1, J4.12 (Pin_12), Q2.3 (D), U6.1 (VBAT)
- new net BOOT0: J1.2 (Pin_2), U6.44 (BOOT0)
- new net BOOT1: J1.5 (Pin_5), U6.20 (PB2/BOOT1)
- new net MIC1: RV1.2, U6.10 (PA0/WKUP/ADC0), U7.1
- new net MIC2: RV2.2, U6.11 (PA1/ADC1), U7.7
- new net OPAMP1: C10.2, J4.9 (Pin_9), U7.3 (+)
- new net OPAMP2: C15.2, J4.10 (Pin_10), U7.5 (+)
- new net PB10: J4.3 (Pin_3), U6.21 (PB10)
- new net PB11: J4.4 (Pin_4), U6.22 (PB11)
- new net PB12: J4.5 (Pin_5), U6.25 (PB12)
- new net PB13: J4.6 (Pin_6), U6.26 (PB13)
- new net PB14: J4.7 (Pin_7), U6.27 (PB14)
- new net PB15: J4.8 (Pin_8), U6.28 (PB15)
- new net RESET: J2.5 (Pin_5), U6.7 (NRST)
- new net USB1_DN: R9.2, U6.32 (PA11/USB1DM)
- new net USB1_DP: R8.2, U6.33 (PA12/USB1DP)
- new net USB2_DN: R13.2, U6.42 (PB6/USB2DM)
- new net USB2_DP: R14.2, U6.43 (PB7/USB2DP)
- no-connect marks 3 -> 10
Other:
- note added: "3.3V SWDIO SWCLK GND RST GND TX RX"
- note added: "TC-6615"
- note removed: "3.3V SWDIO GND RST TX RX"
- moved on the sheet: BT1, C5, C6, D1, J3, JP1, R1, R2, R3, R4, R5, R6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
